Commit message: update

File: urdf/hhfc/urdf/hhfc.urdf (robot description, URDF)
Before this commit: robot hhfc_sf, 15 links, 14 joints
Links:
- link Lleg_ankle_r: geometry collision mesh filename=package://bitbot_gz/urdf/hhfc/meshes/whole_foot_visual.stl; visual mesh filename=package://bitbot_gz/urdf/hhfc/meshes/whole_foot_visual.stl
- link Rleg_ankle_r: geometry collision mesh filename=package://bitbot_gz/urdf/hhfc/meshes/whole_foot_visual.stl; visual mesh filename=package://bitbot_gz/urdf/hhfc/meshes/whole_foot_visual.stl

Commit message: add camera

File: urdf/hhfc/urdf/hhfc.urdf (robot description, URDF)
Before this commit: robot hhfc_sf, 15 links, 14 joints
Links:
- added link camera_link, mass 0.1; visual box size=0.02 0.1 0.02
Joints:
- added joint camera_joint: type fixed, parent base_thorax, child camera_link, origin xyz=0.1 0.0 0.0 rpy=0 0.3490658503988659 0, axis 0 1 0, limit lower=-3.14 upper=3.14 effort=100.0 velocity=100.0

Commit message: update

File: urdf/hhfc/urdf/hhfc.urdf (robot description, URDF)
Before this commit: robot hhfc, 16 links, 15 joints
Links:
- added link lidar_link, mass 0.2; collision cylinder length=0.05 radius=0.03; visual cylinder length=0.05 radius=0.03
- link Lleg_ankle_r: geometry collision mesh filename=package://bitbot_gz/urdf/hhfc/meshes/flat_foot_convex.stl; visual mesh filename=package://bitbot_gz/urdf/hhfc/meshes/flat_foot.stl
- link Rleg_ankle_r: geometry collision mesh filename=package://bitbot_gz/urdf/hhfc/meshes/flat_foot_convex.stl; visual mesh filename=package://bitbot_gz/urdf/hhfc/meshes/flat_foot.stl
Joints:
- added joint lidar_joint: type fixed, parent base_thorax, child lidar_link, origin xyz=0.1 0 0.5 rpy=0 0 0
